File: rgb-plate/rgb-plate.kicad_pcb (KiCad board)
At the start: 2 copper layers, 0 parts

Commit message: initial layout on single board, may need to split up
Parts:
- added C1: 0.1uF, Capacitor_SMD:C_0603_1608Metric, F.Cu at (145.2, 121.0)
- added C10: 10uF, Capacitor_SMD:C_1206_3216Metric, F.Cu at (150.3, 125.4)
- added C11: 0.1uF, Capacitor_SMD:C_0603_1608Metric, F.Cu at (145.2, 131.0)
- added C12: 22uF, Capacitor_SMD:C_1206_3216Metric, F.Cu at (150.3, 128.8)
- added C13: 22uF, Capacitor_SMD:C_1206_3216Metric, F.Cu at (150.3, 132.1)
- added C14: 10nF, Capacitor_SMD:C_0603_1608Metric, F.Cu at (155.9, 111.2)
- added C2: 10uF, Capacitor_SMD:C_1206_3216Metric, F.Cu at (150.3, 108.7)
- added C3: 10uF, Capacitor_SMD:C_1206_3216Metric, F.Cu at (150.3, 112.0)
- added C4: 0.1uF, Capacitor_SMD:C_0603_1608Metric, F.Cu at (145.2, 123.5)
- added C5: 22uF, Capacitor_SMD:C_1206_3216Metric, F.Cu at (150.3, 115.3)
- added C6: 22uF, Capacitor_SMD:C_1206_3216Metric, F.Cu at (150.3, 118.7)
- added C7: 10nF, Capacitor_SMD:C_0603_1608Metric, F.Cu at (145.2, 126.0)
- added C8: 0.1uF, Capacitor_SMD:C_0603_1608Metric, F.Cu at (145.2, 128.5)
- added C9: 10uF, Capacitor_SMD:C_1206_3216Metric, F.Cu at (150.3, 122.0)
- added D1: LED_RGB, LRTBGVSR-4U4V-JW+8A8B-D8-3S4U-7Z:LRTBGVSR4U4VJW8A8BD83S4U7Z, B.Cu at (58.6, 70.6)
- added D10: LED_RGB, LRTBGVSR-4U4V-JW+8A8B-D8-3S4U-7Z:LRTBGVSR4U4VJW8A8BD83S4U7Z, B.Cu at (58.6, 115.6)
- added D100: LED_RGB, LRTBGVSR-4U4V-JW+8A8B-D8-3S4U-7Z:LRTBGVSR4U4VJW8A8BD83S4U7Z, B.Cu at (88.6, 85.6)
- added D101: LED_RGB, LRTBGVSR-4U4V-JW+8A8B-D8-3S4U-7Z:LRTBGVSR4U4VJW8A8BD83S4U7Z, B.Cu at (88.6, 90.6)
- added D102: LED_RGB, LRTBGVSR-4U4V-JW+8A8B-D8-3S4U-7Z:LRTBGVSR4U4VJW8A8BD83S4U7Z, B.Cu at (88.6, 95.6)
- added D103: LED_RGB, LRTBGVSR-4U4V-JW+8A8B-D8-3S4U-7Z:LRTBGVSR4U4VJW8A8BD83S4U7Z, B.Cu at (88.6, 100.6)
- added D104: LED_RGB, LRTBGVSR-4U4V-JW+8A8B-D8-3S4U-7Z:LRTBGVSR4U4VJW8A8BD83S4U7Z, B.Cu at (88.6, 105.6)
- added D105: LED_RGB, LRTBGVSR-4U4V-JW+8A8B-D8-3S4U-7Z:LRTBGVSR4U4VJW8A8BD83S4U7Z, B.Cu at (88.6, 110.6)
- added D106: LED_RGB, LRTBGVSR-4U4V-JW+8A8B-D8-3S4U-7Z:LRTBGVSR4U4VJW8A8BD83S4U7Z, B.Cu at (88.6, 115.6)
- added D107: LED_RGB, LRTBGVSR-4U4V-JW+8A8B-D8-3S4U-7Z:LRTBGVSR4U4VJW8A8BD83S4U7Z, B.Cu at (88.6, 120.6)
- added D108: LED_RGB, LRTBGVSR-4U4V-JW+8A8B-D8-3S4U-7Z:LRTBGVSR4U4VJW8A8BD83S4U7Z, B.Cu at (88.6, 125.6)
- added D109: LED_RGB, LRTBGVSR-4U4V-JW+8A8B-D8-3S4U-7Z:LRTBGVSR4U4VJW8A8BD83S4U7Z, B.Cu at (88.6, 130.6)
- added D11: LED_RGB, LRTBGVSR-4U4V-JW+8A8B-D8-3S4U-7Z:LRTBGVSR4U4VJW8A8BD83S4U7Z, B.Cu at (58.6, 120.6)
- added D110: LED_RGB, LRTBGVSR-4U4V-JW+8A8B-D8-3S4U-7Z:LRTBGVSR4U4VJW8A8BD83S4U7Z, B.Cu at (88.6, 135.6)
- added D111: LED_RGB, LRTBGVSR-4U4V-JW+8A8B-D8-3S4U-7Z:LRTBGVSR4U4VJW8A8BD83S4U7Z, B.Cu at (88.6, 140.6)
- added D112: LED_RGB, LRTBGVSR-4U4V-JW+8A8B-D8-3S4U-7Z:LRTBGVSR4U4VJW8A8BD83S4U7Z, B.Cu at (88.6, 145.6)
- added D113: LED_RGB, LRTBGVSR-4U4V-JW+8A8B-D8-3S4U-7Z:LRTBGVSR4U4VJW8A8BD83S4U7Z, B.Cu at (93.6, 70.6)
- added D114: LED_RGB, LRTBGVSR-4U4V-JW+8A8B-D8-3S4U-7Z:LRTBGVSR4U4VJW8A8BD83S4U7Z, B.Cu at (93.6, 75.6)
- added D115: LED_RGB, LRTBGVSR-4U4V-JW+8A8B-D8-3S4U-7Z:LRTBGVSR4U4VJW8A8BD83S4U7Z, B.Cu at (93.6, 80.6)
- added D116: LED_RGB, LRTBGVSR-4U4V-JW+8A8B-D8-3S4U-7Z:LRTBGVSR4U4VJW8A8BD83S4U7Z, B.Cu at (93.6, 85.6)
- added D117: LED_RGB, LRTBGVSR-4U4V-JW+8A8B-D8-3S4U-7Z:LRTBGVSR4U4VJW8A8BD83S4U7Z, B.Cu at (93.6, 90.6)
- added D118: LED_RGB, LRTBGVSR-4U4V-JW+8A8B-D8-3S4U-7Z:LRTBGVSR4U4VJW8A8BD83S4U7Z, B.Cu at (93.6, 95.6)
- added D119: LED_RGB, LRTBGVSR-4U4V-JW+8A8B-D8-3S4U-7Z:LRTBGVSR4U4VJW8A8BD83S4U7Z, B.Cu at (93.6, 100.6)
- added D12: LED_RGB, LRTBGVSR-4U4V-JW+8A8B-D8-3S4U-7Z:LRTBGVSR4U4VJW8A8BD83S4U7Z, B.Cu at (58.6, 125.6)
- added D120: LED_RGB, LRTBGVSR-4U4V-JW+8A8B-D8-3S4U-7Z:LRTBGVSR4U4VJW8A8BD83S4U7Z, B.Cu at (93.6, 105.6)
- added D121: LED_RGB, LRTBGVSR-4U4V-JW+8A8B-D8-3S4U-7Z:LRTBGVSR4U4VJW8A8BD83S4U7Z, B.Cu at (93.6, 110.6)
- added D122: LED_RGB, LRTBGVSR-4U4V-JW+8A8B-D8-3S4U-7Z:LRTBGVSR4U4VJW8A8BD83S4U7Z, B.Cu at (93.6, 115.6)
- added D123: LED_RGB, LRTBGVSR-4U4V-JW+8A8B-D8-3S4U-7Z:LRTBGVSR4U4VJW8A8BD83S4U7Z, B.Cu at (93.6, 120.6)
- added D124: LED_RGB, LRTBGVSR-4U4V-JW+8A8B-D8-3S4U-7Z:LRTBGVSR4U4VJW8A8BD83S4U7Z, B.Cu at (93.6, 125.6)
- added D125: LED_RGB, LRTBGVSR-4U4V-JW+8A8B-D8-3S4U-7Z:LRTBGVSR4U4VJW8A8BD83S4U7Z, B.Cu at (93.6, 130.6)
- added D126: LED_RGB, LRTBGVSR-4U4V-JW+8A8B-D8-3S4U-7Z:LRTBGVSR4U4VJW8A8BD83S4U7Z, B.Cu at (93.6, 135.6)
- added D127: LED_RGB, LRTBGVSR-4U4V-JW+8A8B-D8-3S4U-7Z:LRTBGVSR4U4VJW8A8BD83S4U7Z, B.Cu at (93.6, 140.6)
- added D128: LED_RGB, LRTBGVSR-4U4V-JW+8A8B-D8-3S4U-7Z:LRTBGVSR4U4VJW8A8BD83S4U7Z, B.Cu at (93.6, 145.6)
- added D129: LED_RGB, LRTBGVSR-4U4V-JW+8A8B-D8-3S4U-7Z:LRTBGVSR4U4VJW8A8BD83S4U7Z, B.Cu at (98.6, 70.6)
- added D13: LED_RGB, LRTBGVSR-4U4V-JW+8A8B-D8-3S4U-7Z:LRTBGVSR4U4VJW8A8BD83S4U7Z, B.Cu at (58.6, 130.6)
- added D130: LED_RGB, LRTBGVSR-4U4V-JW+8A8B-D8-3S4U-7Z:LRTBGVSR4U4VJW8A8BD83S4U7Z, B.Cu at (98.6, 75.6)
- added D131: LED_RGB, LRTBGVSR-4U4V-JW+8A8B-D8-3S4U-7Z:LRTBGVSR4U4VJW8A8BD83S4U7Z, B.Cu at (98.6, 80.6)
- added D132: LED_RGB, LRTBGVSR-4U4V-JW+8A8B-D8-3S4U-7Z:LRTBGVSR4U4VJW8A8BD83S4U7Z, B.Cu at (98.6, 85.6)
- added D133: LED_RGB, LRTBGVSR-4U4V-JW+8A8B-D8-3S4U-7Z:LRTBGVSR4U4VJW8A8BD83S4U7Z, B.Cu at (98.6, 90.6)
- added D134: LED_RGB, LRTBGVSR-4U4V-JW+8A8B-D8-3S4U-7Z:LRTBGVSR4U4VJW8A8BD83S4U7Z, B.Cu at (98.6, 95.6)
- added D135: LED_RGB, LRTBGVSR-4U4V-JW+8A8B-D8-3S4U-7Z:LRTBGVSR4U4VJW8A8BD83S4U7Z, B.Cu at (98.6, 100.6)
- added D136: LED_RGB, LRTBGVSR-4U4V-JW+8A8B-D8-3S4U-7Z:LRTBGVSR4U4VJW8A8BD83S4U7Z, B.Cu at (98.6, 105.6)
- added D137: LED_RGB, LRTBGVSR-4U4V-JW+8A8B-D8-3S4U-7Z:LRTBGVSR4U4VJW8A8BD83S4U7Z, B.Cu at (98.6, 110.6)
- added D138: LED_RGB, LRTBGVSR-4U4V-JW+8A8B-D8-3S4U-7Z:LRTBGVSR4U4VJW8A8BD83S4U7Z, B.Cu at (98.6, 115.6)
- added D139: LED_RGB, LRTBGVSR-4U4V-JW+8A8B-D8-3S4U-7Z:LRTBGVSR4U4VJW8A8BD83S4U7Z, B.Cu at (98.6, 120.6)
- added D14: LED_RGB, LRTBGVSR-4U4V-JW+8A8B-D8-3S4U-7Z:LRTBGVSR4U4VJW8A8BD83S4U7Z, B.Cu at (58.6, 135.6)
- added D140: LED_RGB, LRTBGVSR-4U4V-JW+8A8B-D8-3S4U-7Z:LRTBGVSR4U4VJW8A8BD83S4U7Z, B.Cu at (98.6, 125.6)
- added D141: LED_RGB, LRTBGVSR-4U4V-JW+8A8B-D8-3S4U-7Z:LRTBGVSR4U4VJW8A8BD83S4U7Z, B.Cu at (98.6, 130.6)
- added D142: LED_RGB, LRTBGVSR-4U4V-JW+8A8B-D8-3S4U-7Z:LRTBGVSR4U4VJW8A8BD83S4U7Z, B.Cu at (98.6, 135.6)
- added D143: LED_RGB, LRTBGVSR-4U4V-JW+8A8B-D8-3S4U-7Z:LRTBGVSR4U4VJW8A8BD83S4U7Z, B.Cu at (98.6, 140.6)
- added D144: LED_RGB, LRTBGVSR-4U4V-JW+8A8B-D8-3S4U-7Z:LRTBGVSR4U4VJW8A8BD83S4U7Z, B.Cu at (98.6, 145.6)
- added D145: LED_RGB, LRTBGVSR-4U4V-JW+8A8B-D8-3S4U-7Z:LRTBGVSR4U4VJW8A8BD83S4U7Z, B.Cu at (103.6, 70.6)
- added D146: LED_RGB, LRTBGVSR-4U4V-JW+8A8B-D8-3S4U-7Z:LRTBGVSR4U4VJW8A8BD83S4U7Z, B.Cu at (103.6, 75.6)
- added D147: LED_RGB, LRTBGVSR-4U4V-JW+8A8B-D8-3S4U-7Z:LRTBGVSR4U4VJW8A8BD83S4U7Z, B.Cu at (103.6, 80.6)
- added D148: LED_RGB, LRTBGVSR-4U4V-JW+8A8B-D8-3S4U-7Z:LRTBGVSR4U4VJW8A8BD83S4U7Z, B.Cu at (103.6, 85.6)
- added D149: LED_RGB, LRTBGVSR-4U4V-JW+8A8B-D8-3S4U-7Z:LRTBGVSR4U4VJW8A8BD83S4U7Z, B.Cu at (103.6, 90.6)
- added D15: LED_RGB, LRTBGVSR-4U4V-JW+8A8B-D8-3S4U-7Z:LRTBGVSR4U4VJW8A8BD83S4U7Z, B.Cu at (58.6, 140.6)
- added D150: LED_RGB, LRTBGVSR-4U4V-JW+8A8B-D8-3S4U-7Z:LRTBGVSR4U4VJW8A8BD83S4U7Z, B.Cu at (103.6, 95.6)
- added D151: LED_RGB, LRTBGVSR-4U4V-JW+8A8B-D8-3S4U-7Z:LRTBGVSR4U4VJW8A8BD83S4U7Z, B.Cu at (103.6, 100.6)
- added D152: LED_RGB, LRTBGVSR-4U4V-JW+8A8B-D8-3S4U-7Z:LRTBGVSR4U4VJW8A8BD83S4U7Z, B.Cu at (103.6, 105.6)
- added D153: LED_RGB, LRTBGVSR-4U4V-JW+8A8B-D8-3S4U-7Z:LRTBGVSR4U4VJW8A8BD83S4U7Z, B.Cu at (103.6, 110.6)
- added D154: LED_RGB, LRTBGVSR-4U4V-JW+8A8B-D8-3S4U-7Z:LRTBGVSR4U4VJW8A8BD83S4U7Z, B.Cu at (103.6, 115.6)
- added D155: LED_RGB, LRTBGVSR-4U4V-JW+8A8B-D8-3S4U-7Z:LRTBGVSR4U4VJW8A8BD83S4U7Z, B.Cu at (103.6, 120.6)
- added D156: LED_RGB, LRTBGVSR-4U4V-JW+8A8B-D8-3S4U-7Z:LRTBGVSR4U4VJW8A8BD83S4U7Z, B.Cu at (103.6, 125.6)
- added D157: LED_RGB, LRTBGVSR-4U4V-JW+8A8B-D8-3S4U-7Z:LRTBGVSR4U4VJW8A8BD83S4U7Z, B.Cu at (103.6, 130.6)
- added D158: LED_RGB, LRTBGVSR-4U4V-JW+8A8B-D8-3S4U-7Z:LRTBGVSR4U4VJW8A8BD83S4U7Z, B.Cu at (103.6, 135.6)
- added D159: LED_RGB, LRTBGVSR-4U4V-JW+8A8B-D8-3S4U-7Z:LRTBGVSR4U4VJW8A8BD83S4U7Z, B.Cu at (103.6, 140.6)
- added D16: LED_RGB, LRTBGVSR-4U4V-JW+8A8B-D8-3S4U-7Z:LRTBGVSR4U4VJW8A8BD83S4U7Z, B.Cu at (58.6, 145.6)
- added D160: LED_RGB, LRTBGVSR-4U4V-JW+8A8B-D8-3S4U-7Z:LRTBGVSR4U4VJW8A8BD83S4U7Z, B.Cu at (103.6, 145.6)
- added D161: LED_RGB, LRTBGVSR-4U4V-JW+8A8B-D8-3S4U-7Z:LRTBGVSR4U4VJW8A8BD83S4U7Z, B.Cu at (108.6, 70.6)
- added D162: LED_RGB, LRTBGVSR-4U4V-JW+8A8B-D8-3S4U-7Z:LRTBGVSR4U4VJW8A8BD83S4U7Z, B.Cu at (108.6, 75.6)
- added D163: LED_RGB, LRTBGVSR-4U4V-JW+8A8B-D8-3S4U-7Z:LRTBGVSR4U4VJW8A8BD83S4U7Z, B.Cu at (108.6, 80.6)
- added D164: LED_RGB, LRTBGVSR-4U4V-JW+8A8B-D8-3S4U-7Z:LRTBGVSR4U4VJW8A8BD83S4U7Z, B.Cu at (108.6, 85.6)
- added D165: LED_RGB, LRTBGVSR-4U4V-JW+8A8B-D8-3S4U-7Z:LRTBGVSR4U4VJW8A8BD83S4U7Z, B.Cu at (108.6, 90.6)
- added D166: LED_RGB, LRTBGVSR-4U4V-JW+8A8B-D8-3S4U-7Z:LRTBGVSR4U4VJW8A8BD83S4U7Z, B.Cu at (108.6, 95.6)
- added D167: LED_RGB, LRTBGVSR-4U4V-JW+8A8B-D8-3S4U-7Z:LRTBGVSR4U4VJW8A8BD83S4U7Z, B.Cu at (108.6, 100.6)
- added D168: LED_RGB, LRTBGVSR-4U4V-JW+8A8B-D8-3S4U-7Z:LRTBGVSR4U4VJW8A8BD83S4U7Z, B.Cu at (108.6, 105.6)
- added D169: LED_RGB, LRTBGVSR-4U4V-JW+8A8B-D8-3S4U-7Z:LRTBGVSR4U4VJW8A8BD83S4U7Z, B.Cu at (108.6, 110.6)
- added D17: LED_RGB, LRTBGVSR-4U4V-JW+8A8B-D8-3S4U-7Z:LRTBGVSR4U4VJW8A8BD83S4U7Z, B.Cu at (63.6, 70.6)
- added D170: LED_RGB, LRTBGVSR-4U4V-JW+8A8B-D8-3S4U-7Z:LRTBGVSR4U4VJW8A8BD83S4U7Z, B.Cu at (108.6, 115.6)
- added D171: LED_RGB, LRTBGVSR-4U4V-JW+8A8B-D8-3S4U-7Z:LRTBGVSR4U4VJW8A8BD83S4U7Z, B.Cu at (108.6, 120.6)
- added D172: LED_RGB, LRTBGVSR-4U4V-JW+8A8B-D8-3S4U-7Z:LRTBGVSR4U4VJW8A8BD83S4U7Z, B.Cu at (108.6, 125.6)
- added D173: LED_RGB, LRTBGVSR-4U4V-JW+8A8B-D8-3S4U-7Z:LRTBGVSR4U4VJW8A8BD83S4U7Z, B.Cu at (108.6, 130.6)
- added D174: LED_RGB, LRTBGVSR-4U4V-JW+8A8B-D8-3S4U-7Z:LRTBGVSR4U4VJW8A8BD83S4U7Z, B.Cu at (108.6, 135.6)
- added D175: LED_RGB, LRTBGVSR-4U4V-JW+8A8B-D8-3S4U-7Z:LRTBGVSR4U4VJW8A8BD83S4U7Z, B.Cu at (108.6, 140.6)
- added D176: LED_RGB, LRTBGVSR-4U4V-JW+8A8B-D8-3S4U-7Z:LRTBGVSR4U4VJW8A8BD83S4U7Z, B.Cu at (108.6, 145.6)
- added D177: LED_RGB, LRTBGVSR-4U4V-JW+8A8B-D8-3S4U-7Z:LRTBGVSR4U4VJW8A8BD83S4U7Z, B.Cu at (113.6, 70.6)
- added D178: LED_RGB, LRTBGVSR-4U4V-JW+8A8B-D8-3S4U-7Z:LRTBGVSR4U4VJW8A8BD83S4U7Z, B.Cu at (113.6, 75.6)
- added D179: LED_RGB, LRTBGVSR-4U4V-JW+8A8B-D8-3S4U-7Z:LRTBGVSR4U4VJW8A8BD83S4U7Z, B.Cu at (113.6, 80.6)
- added D18: LED_RGB, LRTBGVSR-4U4V-JW+8A8B-D8-3S4U-7Z:LRTBGVSR4U4VJW8A8BD83S4U7Z, B.Cu at (63.6, 75.6)
- added D180: LED_RGB, LRTBGVSR-4U4V-JW+8A8B-D8-3S4U-7Z:LRTBGVSR4U4VJW8A8BD83S4U7Z, B.Cu at (113.6, 85.6)
- added D181: LED_RGB, LRTBGVSR-4U4V-JW+8A8B-D8-3S4U-7Z:LRTBGVSR4U4VJW8A8BD83S4U7Z, B.Cu at (113.6, 90.6)
- added D182: LED_RGB, LRTBGVSR-4U4V-JW+8A8B-D8-3S4U-7Z:LRTBGVSR4U4VJW8A8BD83S4U7Z, B.Cu at (113.6, 95.6)
- added D183: LED_RGB, LRTBGVSR-4U4V-JW+8A8B-D8-3S4U-7Z:LRTBGVSR4U4VJW8A8BD83S4U7Z, B.Cu at (113.6, 100.6)
- added D184: LED_RGB, LRTBGVSR-4U4V-JW+8A8B-D8-3S4U-7Z:LRTBGVSR4U4VJW8A8BD83S4U7Z, B.Cu at (113.6, 105.6)
- added D185: LED_RGB, LRTBGVSR-4U4V-JW+8A8B-D8-3S4U-7Z:LRTBGVSR4U4VJW8A8BD83S4U7Z, B.Cu at (113.6, 110.6)
- added D186: LED_RGB, LRTBGVSR-4U4V-JW+8A8B-D8-3S4U-7Z:LRTBGVSR4U4VJW8A8BD83S4U7Z, B.Cu at (113.6, 115.6)
- added D187: LED_RGB, LRTBGVSR-4U4V-JW+8A8B-D8-3S4U-7Z:LRTBGVSR4U4VJW8A8BD83S4U7Z, B.Cu at (113.6, 120.6)
- added D188: LED_RGB, LRTBGVSR-4U4V-JW+8A8B-D8-3S4U-7Z:LRTBGVSR4U4VJW8A8BD83S4U7Z, B.Cu at (113.6, 125.6)
- added D189: LED_RGB, LRTBGVSR-4U4V-JW+8A8B-D8-3S4U-7Z:LRTBGVSR4U4VJW8A8BD83S4U7Z, B.Cu at (113.6, 130.6)
- added D19: LED_RGB, LRTBGVSR-4U4V-JW+8A8B-D8-3S4U-7Z:LRTBGVSR4U4VJW8A8BD83S4U7Z, B.Cu at (63.6, 80.6)
- added D190: LED_RGB, LRTBGVSR-4U4V-JW+8A8B-D8-3S4U-7Z:LRTBGVSR4U4VJW8A8BD83S4U7Z, B.Cu at (113.6, 135.6)
- added D191: LED_RGB, LRTBGVSR-4U4V-JW+8A8B-D8-3S4U-7Z:LRTBGVSR4U4VJW8A8BD83S4U7Z, B.Cu at (113.6, 140.6)
- added D192: LED_RGB, LRTBGVSR-4U4V-JW+8A8B-D8-3S4U-7Z:LRTBGVSR4U4VJW8A8BD83S4U7Z, B.Cu at (113.6, 145.6)
- added D193: LED_RGB, LRTBGVSR-4U4V-JW+8A8B-D8-3S4U-7Z:LRTBGVSR4U4VJW8A8BD83S4U7Z, B.Cu at (118.6, 70.6)
- added D194: LED_RGB, LRTBGVSR-4U4V-JW+8A8B-D8-3S4U-7Z:LRTBGVSR4U4VJW8A8BD83S4U7Z, B.Cu at (118.6, 75.6)
- added D195: LED_RGB, LRTBGVSR-4U4V-JW+8A8B-D8-3S4U-7Z:LRTBGVSR4U4VJW8A8BD83S4U7Z, B.Cu at (118.6, 80.6)
- added D196: LED_RGB, LRTBGVSR-4U4V-JW+8A8B-D8-3S4U-7Z:LRTBGVSR4U4VJW8A8BD83S4U7Z, B.Cu at (118.6, 85.6)
- added D197: LED_RGB, LRTBGVSR-4U4V-JW+8A8B-D8-3S4U-7Z:LRTBGVSR4U4VJW8A8BD83S4U7Z, B.Cu at (118.6, 90.6)
- added D198: LED_RGB, LRTBGVSR-4U4V-JW+8A8B-D8-3S4U-7Z:LRTBGVSR4U4VJW8A8BD83S4U7Z, B.Cu at (118.6, 95.6)
- added D199: LED_RGB, LRTBGVSR-4U4V-JW+8A8B-D8-3S4U-7Z:LRTBGVSR4U4VJW8A8BD83S4U7Z, B.Cu at (118.6, 100.6)
- added D2: LED_RGB, LRTBGVSR-4U4V-JW+8A8B-D8-3S4U-7Z:LRTBGVSR4U4VJW8A8BD83S4U7Z, B.Cu at (58.6, 75.6)
- added D20: LED_RGB, LRTBGVSR-4U4V-JW+8A8B-D8-3S4U-7Z:LRTBGVSR4U4VJW8A8BD83S4U7Z, B.Cu at (63.6, 85.6)
- added D200: LED_RGB, LRTBGVSR-4U4V-JW+8A8B-D8-3S4U-7Z:LRTBGVSR4U4VJW8A8BD83S4U7Z, B.Cu at (118.6, 105.6)
- added D201: LED_RGB, LRTBGVSR-4U4V-JW+8A8B-D8-3S4U-7Z:LRTBGVSR4U4VJW8A8BD83S4U7Z, B.Cu at (118.6, 110.6)
- added D202: LED_RGB, LRTBGVSR-4U4V-JW+8A8B-D8-3S4U-7Z:LRTBGVSR4U4VJW8A8BD83S4U7Z, B.Cu at (118.6, 115.6)
- added D203: LED_RGB, LRTBGVSR-4U4V-JW+8A8B-D8-3S4U-7Z:LRTBGVSR4U4VJW8A8BD83S4U7Z, B.Cu at (118.6, 120.6)
- added D204: LED_RGB, LRTBGVSR-4U4V-JW+8A8B-D8-3S4U-7Z:LRTBGVSR4U4VJW8A8BD83S4U7Z, B.Cu at (118.6, 125.6)
- added D205: LED_RGB, LRTBGVSR-4U4V-JW+8A8B-D8-3S4U-7Z:LRTBGVSR4U4VJW8A8BD83S4U7Z, B.Cu at (118.6, 130.6)
- added D206: LED_RGB, LRTBGVSR-4U4V-JW+8A8B-D8-3S4U-7Z:LRTBGVSR4U4VJW8A8BD83S4U7Z, B.Cu at (118.6, 135.6)
- added D207: LED_RGB, LRTBGVSR-4U4V-JW+8A8B-D8-3S4U-7Z:LRTBGVSR4U4VJW8A8BD83S4U7Z, B.Cu at (118.6, 140.6)
- added D208: LED_RGB, LRTBGVSR-4U4V-JW+8A8B-D8-3S4U-7Z:LRTBGVSR4U4VJW8A8BD83S4U7Z, B.Cu at (118.6, 145.6)
- added D209: LED_RGB, LRTBGVSR-4U4V-JW+8A8B-D8-3S4U-7Z:LRTBGVSR4U4VJW8A8BD83S4U7Z, B.Cu at (123.6, 70.6)
- added D21: LED_RGB, LRTBGVSR-4U4V-JW+8A8B-D8-3S4U-7Z:LRTBGVSR4U4VJW8A8BD83S4U7Z, B.Cu at (63.6, 90.6)
- added D210: LED_RGB, LRTBGVSR-4U4V-JW+8A8B-D8-3S4U-7Z:LRTBGVSR4U4VJW8A8BD83S4U7Z, B.Cu at (123.6, 75.6)
- added D211: LED_RGB, LRTBGVSR-4U4V-JW+8A8B-D8-3S4U-7Z:LRTBGVSR4U4VJW8A8BD83S4U7Z, B.Cu at (123.6, 80.6)
- added D212: LED_RGB, LRTBGVSR-4U4V-JW+8A8B-D8-3S4U-7Z:LRTBGVSR4U4VJW8A8BD83S4U7Z, B.Cu at (123.6, 85.6)
- added D213: LED_RGB, LRTBGVSR-4U4V-JW+8A8B-D8-3S4U-7Z:LRTBGVSR4U4VJW8A8BD83S4U7Z, B.Cu at (123.6, 90.6)
- added D214: LED_RGB, LRTBGVSR-4U4V-JW+8A8B-D8-3S4U-7Z:LRTBGVSR4U4VJW8A8BD83S4U7Z, B.Cu at (123.6, 95.6)
- added D215: LED_RGB, LRTBGVSR-4U4V-JW+8A8B-D8-3S4U-7Z:LRTBGVSR4U4VJW8A8BD83S4U7Z, B.Cu at (123.6, 100.6)
- added D216: LED_RGB, LRTBGVSR-4U4V-JW+8A8B-D8-3S4U-7Z:LRTBGVSR4U4VJW8A8BD83S4U7Z, B.Cu at (123.6, 105.6)
- added D217: LED_RGB, LRTBGVSR-4U4V-JW+8A8B-D8-3S4U-7Z:LRTBGVSR4U4VJW8A8BD83S4U7Z, B.Cu at (123.6, 110.6)
- added D218: LED_RGB, LRTBGVSR-4U4V-JW+8A8B-D8-3S4U-7Z:LRTBGVSR4U4VJW8A8BD83S4U7Z, B.Cu at (123.6, 115.6)
- added D219: LED_RGB, LRTBGVSR-4U4V-JW+8A8B-D8-3S4U-7Z:LRTBGVSR4U4VJW8A8BD83S4U7Z, B.Cu at (123.6, 120.6)
- added D22: LED_RGB, LRTBGVSR-4U4V-JW+8A8B-D8-3S4U-7Z:LRTBGVSR4U4VJW8A8BD83S4U7Z, B.Cu at (63.6, 95.6)
- added D220: LED_RGB, LRTBGVSR-4U4V-JW+8A8B-D8-3S4U-7Z:LRTBGVSR4U4VJW8A8BD83S4U7Z, B.Cu at (123.6, 125.6)
- added D221: LED_RGB, LRTBGVSR-4U4V-JW+8A8B-D8-3S4U-7Z:LRTBGVSR4U4VJW8A8BD83S4U7Z, B.Cu at (123.6, 130.6)
- added D222: LED_RGB, LRTBGVSR-4U4V-JW+8A8B-D8-3S4U-7Z:LRTBGVSR4U4VJW8A8BD83S4U7Z, B.Cu at (123.6, 135.6)
- added D223: LED_RGB, LRTBGVSR-4U4V-JW+8A8B-D8-3S4U-7Z:LRTBGVSR4U4VJW8A8BD83S4U7Z, B.Cu at (123.6, 140.6)
- added D224: LED_RGB, LRTBGVSR-4U4V-JW+8A8B-D8-3S4U-7Z:LRTBGVSR4U4VJW8A8BD83S4U7Z, B.Cu at (123.6, 145.6)
- added D225: LED_RGB, LRTBGVSR-4U4V-JW+8A8B-D8-3S4U-7Z:LRTBGVSR4U4VJW8A8BD83S4U7Z, B.Cu at (128.6, 70.6)
- added D226: LED_RGB, LRTBGVSR-4U4V-JW+8A8B-D8-3S4U-7Z:LRTBGVSR4U4VJW8A8BD83S4U7Z, B.Cu at (128.6, 75.6)
- added D227: LED_RGB, LRTBGVSR-4U4V-JW+8A8B-D8-3S4U-7Z:LRTBGVSR4U4VJW8A8BD83S4U7Z, B.Cu at (128.6, 80.6)
- added D228: LED_RGB, LRTBGVSR-4U4V-JW+8A8B-D8-3S4U-7Z:LRTBGVSR4U4VJW8A8BD83S4U7Z, B.Cu at (128.6, 85.6)
- added D229: LED_RGB, LRTBGVSR-4U4V-JW+8A8B-D8-3S4U-7Z:LRTBGVSR4U4VJW8A8BD83S4U7Z, B.Cu at (128.6, 90.6)
- added D23: LED_RGB, LRTBGVSR-4U4V-JW+8A8B-D8-3S4U-7Z:LRTBGVSR4U4VJW8A8BD83S4U7Z, B.Cu at (63.6, 100.6)
- added D230: LED_RGB, LRTBGVSR-4U4V-JW+8A8B-D8-3S4U-7Z:LRTBGVSR4U4VJW8A8BD83S4U7Z, B.Cu at (128.6, 95.6)
- added D231: LED_RGB, LRTBGVSR-4U4V-JW+8A8B-D8-3S4U-7Z:LRTBGVSR4U4VJW8A8BD83S4U7Z, B.Cu at (128.6, 100.6)
- added D232: LED_RGB, LRTBGVSR-4U4V-JW+8A8B-D8-3S4U-7Z:LRTBGVSR4U4VJW8A8BD83S4U7Z, B.Cu at (128.6, 105.6)
- added D233: LED_RGB, LRTBGVSR-4U4V-JW+8A8B-D8-3S4U-7Z:LRTBGVSR4U4VJW8A8BD83S4U7Z, B.Cu at (128.6, 110.6)
- added D234: LED_RGB, LRTBGVSR-4U4V-JW+8A8B-D8-3S4U-7Z:LRTBGVSR4U4VJW8A8BD83S4U7Z, B.Cu at (128.6, 115.6)
- added D235: LED_RGB, LRTBGVSR-4U4V-JW+8A8B-D8-3S4U-7Z:LRTBGVSR4U4VJW8A8BD83S4U7Z, B.Cu at (128.6, 120.6)
- added D236: LED_RGB, LRTBGVSR-4U4V-JW+8A8B-D8-3S4U-7Z:LRTBGVSR4U4VJW8A8BD83S4U7Z, B.Cu at (128.6, 125.6)
- added D237: LED_RGB, LRTBGVSR-4U4V-JW+8A8B-D8-3S4U-7Z:LRTBGVSR4U4VJW8A8BD83S4U7Z, B.Cu at (128.6, 130.6)
- added D238: LED_RGB, LRTBGVSR-4U4V-JW+8A8B-D8-3S4U-7Z:LRTBGVSR4U4VJW8A8BD83S4U7Z, B.Cu at (128.6, 135.6)
- added D239: LED_RGB, LRTBGVSR-4U4V-JW+8A8B-D8-3S4U-7Z:LRTBGVSR4U4VJW8A8BD83S4U7Z, B.Cu at (128.6, 140.6)
- added D24: LED_RGB, LRTBGVSR-4U4V-JW+8A8B-D8-3S4U-7Z:LRTBGVSR4U4VJW8A8BD83S4U7Z, B.Cu at (63.6, 105.6)
- added D240: LED_RGB, LRTBGVSR-4U4V-JW+8A8B-D8-3S4U-7Z:LRTBGVSR4U4VJW8A8BD83S4U7Z, B.Cu at (128.6, 145.6)
- added D241: LED_RGB, LRTBGVSR-4U4V-JW+8A8B-D8-3S4U-7Z:LRTBGVSR4U4VJW8A8BD83S4U7Z, B.Cu at (133.6, 70.6)
- added D242: LED_RGB, LRTBGVSR-4U4V-JW+8A8B-D8-3S4U-7Z:LRTBGVSR4U4VJW8A8BD83S4U7Z, B.Cu at (133.6, 75.6)
- added D243: LED_RGB, LRTBGVSR-4U4V-JW+8A8B-D8-3S4U-7Z:LRTBGVSR4U4VJW8A8BD83S4U7Z, B.Cu at (133.6, 80.6)
- added D244: LED_RGB, LRTBGVSR-4U4V-JW+8A8B-D8-3S4U-7Z:LRTBGVSR4U4VJW8A8BD83S4U7Z, B.Cu at (133.6, 85.6)
- added D245: LED_RGB, LRTBGVSR-4U4V-JW+8A8B-D8-3S4U-7Z:LRTBGVSR4U4VJW8A8BD83S4U7Z, B.Cu at (133.6, 90.6)
- added D246: LED_RGB, LRTBGVSR-4U4V-JW+8A8B-D8-3S4U-7Z:LRTBGVSR4U4VJW8A8BD83S4U7Z, B.Cu at (133.6, 95.6)
- added D247: LED_RGB, LRTBGVSR-4U4V-JW+8A8B-D8-3S4U-7Z:LRTBGVSR4U4VJW8A8BD83S4U7Z, B.Cu at (133.6, 100.6)
- added D248: LED_RGB, LRTBGVSR-4U4V-JW+8A8B-D8-3S4U-7Z:LRTBGVSR4U4VJW8A8BD83S4U7Z, B.Cu at (133.6, 105.6)
- added D249: LED_RGB, LRTBGVSR-4U4V-JW+8A8B-D8-3S4U-7Z:LRTBGVSR4U4VJW8A8BD83S4U7Z, B.Cu at (133.6, 110.6)
- added D25: LED_RGB, LRTBGVSR-4U4V-JW+8A8B-D8-3S4U-7Z:LRTBGVSR4U4VJW8A8BD83S4U7Z, B.Cu at (63.6, 110.6)
- added D250: LED_RGB, LRTBGVSR-4U4V-JW+8A8B-D8-3S4U-7Z:LRTBGVSR4U4VJW8A8BD83S4U7Z, B.Cu at (133.6, 115.6)
- added D251: LED_RGB, LRTBGVSR-4U4V-JW+8A8B-D8-3S4U-7Z:LRTBGVSR4U4VJW8A8BD83S4U7Z, B.Cu at (133.6, 120.6)
- added D252: LED_RGB, LRTBGVSR-4U4V-JW+8A8B-D8-3S4U-7Z:LRTBGVSR4U4VJW8A8BD83S4U7Z, B.Cu at (133.6, 125.6)
- added D253: LED_RGB, LRTBGVSR-4U4V-JW+8A8B-D8-3S4U-7Z:LRTBGVSR4U4VJW8A8BD83S4U7Z, B.Cu at (133.6, 130.6)
- added D254: LED_RGB, LRTBGVSR-4U4V-JW+8A8B-D8-3S4U-7Z:LRTBGVSR4U4VJW8A8BD83S4U7Z, B.Cu at (133.6, 135.6)
- added D255: LED_RGB, LRTBGVSR-4U4V-JW+8A8B-D8-3S4U-7Z:LRTBGVSR4U4VJW8A8BD83S4U7Z, B.Cu at (133.6, 140.6)
- added D256: LED_RGB, LRTBGVSR-4U4V-JW+8A8B-D8-3S4U-7Z:LRTBGVSR4U4VJW8A8BD83S4U7Z, B.Cu at (133.6, 145.6)
- added D26: LED_RGB, LRTBGVSR-4U4V-JW+8A8B-D8-3S4U-7Z:LRTBGVSR4U4VJW8A8BD83S4U7Z, B.Cu at (63.6, 115.6)
- added D27: LED_RGB, LRTBGVSR-4U4V-JW+8A8B-D8-3S4U-7Z:LRTBGVSR4U4VJW8A8BD83S4U7Z, B.Cu at (63.6, 120.6)
- added D28: LED_RGB, LRTBGVSR-4U4V-JW+8A8B-D8-3S4U-7Z:LRTBGVSR4U4VJW8A8BD83S4U7Z, B.Cu at (63.6, 125.6)
- added D29: LED_RGB, LRTBGVSR-4U4V-JW+8A8B-D8-3S4U-7Z:LRTBGVSR4U4VJW8A8BD83S4U7Z, B.Cu at (63.6, 130.6)
- added D3: LED_RGB, LRTBGVSR-4U4V-JW+8A8B-D8-3S4U-7Z:LRTBGVSR4U4VJW8A8BD83S4U7Z, B.Cu at (58.6, 80.6)
- added D30: LED_RGB, LRTBGVSR-4U4V-JW+8A8B-D8-3S4U-7Z:LRTBGVSR4U4VJW8A8BD83S4U7Z, B.Cu at (63.6, 135.6)
- added D31: LED_RGB, LRTBGVSR-4U4V-JW+8A8B-D8-3S4U-7Z:LRTBGVSR4U4VJW8A8BD83S4U7Z, B.Cu at (63.6, 140.6)
- added D32: LED_RGB, LRTBGVSR-4U4V-JW+8A8B-D8-3S4U-7Z:LRTBGVSR4U4VJW8A8BD83S4U7Z, B.Cu at (63.6, 145.6)
- added D33: LED_RGB, LRTBGVSR-4U4V-JW+8A8B-D8-3S4U-7Z:LRTBGVSR4U4VJW8A8BD83S4U7Z, B.Cu at (68.6, 70.6)
- added D34: LED_RGB, LRTBGVSR-4U4V-JW+8A8B-D8-3S4U-7Z:LRTBGVSR4U4VJW8A8BD83S4U7Z, B.Cu at (68.6, 75.6)
- added D35: LED_RGB, LRTBGVSR-4U4V-JW+8A8B-D8-3S4U-7Z:LRTBGVSR4U4VJW8A8BD83S4U7Z, B.Cu at (68.6, 80.6)
- added D36: LED_RGB, LRTBGVSR-4U4V-JW+8A8B-D8-3S4U-7Z:LRTBGVSR4U4VJW8A8BD83S4U7Z, B.Cu at (68.6, 85.6)
- added D37: LED_RGB, LRTBGVSR-4U4V-JW+8A8B-D8-3S4U-7Z:LRTBGVSR4U4VJW8A8BD83S4U7Z, B.Cu at (68.6, 90.6)
- added D38: LED_RGB, LRTBGVSR-4U4V-JW+8A8B-D8-3S4U-7Z:LRTBGVSR4U4VJW8A8BD83S4U7Z, B.Cu at (68.6, 95.6)
- added D39: LED_RGB, LRTBGVSR-4U4V-JW+8A8B-D8-3S4U-7Z:LRTBGVSR4U4VJW8A8BD83S4U7Z, B.Cu at (68.6, 100.6)
- added D4: LED_RGB, LRTBGVSR-4U4V-JW+8A8B-D8-3S4U-7Z:LRTBGVSR4U4VJW8A8BD83S4U7Z, B.Cu at (58.6, 85.6)
- added D40: LED_RGB, LRTBGVSR-4U4V-JW+8A8B-D8-3S4U-7Z:LRTBGVSR4U4VJW8A8BD83S4U7Z, B.Cu at (68.6, 105.6)
- added D41: LED_RGB, LRTBGVSR-4U4V-JW+8A8B-D8-3S4U-7Z:LRTBGVSR4U4VJW8A8BD83S4U7Z, B.Cu at (68.6, 110.6)
- added D42: LED_RGB, LRTBGVSR-4U4V-JW+8A8B-D8-3S4U-7Z:LRTBGVSR4U4VJW8A8BD83S4U7Z, B.Cu at (68.6, 115.6)
- added D43: LED_RGB, LRTBGVSR-4U4V-JW+8A8B-D8-3S4U-7Z:LRTBGVSR4U4VJW8A8BD83S4U7Z, B.Cu at (68.6, 120.6)
- added D44: LED_RGB, LRTBGVSR-4U4V-JW+8A8B-D8-3S4U-7Z:LRTBGVSR4U4VJW8A8BD83S4U7Z, B.Cu at (68.6, 125.6)
- added D45: LED_RGB, LRTBGVSR-4U4V-JW+8A8B-D8-3S4U-7Z:LRTBGVSR4U4VJW8A8BD83S4U7Z, B.Cu at (68.6, 130.6)
- added D46: LED_RGB, LRTBGVSR-4U4V-JW+8A8B-D8-3S4U-7Z:LRTBGVSR4U4VJW8A8BD83S4U7Z, B.Cu at (68.6, 135.6)
- added D47: LED_RGB, LRTBGVSR-4U4V-JW+8A8B-D8-3S4U-7Z:LRTBGVSR4U4VJW8A8BD83S4U7Z, B.Cu at (68.6, 140.6)
- added D48: LED_RGB, LRTBGVSR-4U4V-JW+8A8B-D8-3S4U-7Z:LRTBGVSR4U4VJW8A8BD83S4U7Z, B.Cu at (68.6, 145.6)
- added D49: LED_RGB, LRTBGVSR-4U4V-JW+8A8B-D8-3S4U-7Z:LRTBGVSR4U4VJW8A8BD83S4U7Z, B.Cu at (73.6, 70.6)
- added D5: LED_RGB, LRTBGVSR-4U4V-JW+8A8B-D8-3S4U-7Z:LRTBGVSR4U4VJW8A8BD83S4U7Z, B.Cu at (58.6, 90.6)
- added D50: LED_RGB, LRTBGVSR-4U4V-JW+8A8B-D8-3S4U-7Z:LRTBGVSR4U4VJW8A8BD83S4U7Z, B.Cu at (73.6, 75.6)
- added D51: LED_RGB, LRTBGVSR-4U4V-JW+8A8B-D8-3S4U-7Z:LRTBGVSR4U4VJW8A8BD83S4U7Z, B.Cu at (73.6, 80.6)
- added D52: LED_RGB, LRTBGVSR-4U4V-JW+8A8B-D8-3S4U-7Z:LRTBGVSR4U4VJW8A8BD83S4U7Z, B.Cu at (73.6, 85.6)
- added D53: LED_RGB, LRTBGVSR-4U4V-JW+8A8B-D8-3S4U-7Z:LRTBGVSR4U4VJW8A8BD83S4U7Z, B.Cu at (73.6, 90.6)
- added D54: LED_RGB, LRTBGVSR-4U4V-JW+8A8B-D8-3S4U-7Z:LRTBGVSR4U4VJW8A8BD83S4U7Z, B.Cu at (73.6, 95.6)
- added D55: LED_RGB, LRTBGVSR-4U4V-JW+8A8B-D8-3S4U-7Z:LRTBGVSR4U4VJW8A8BD83S4U7Z, B.Cu at (73.6, 100.6)
- added D56: LED_RGB, LRTBGVSR-4U4V-JW+8A8B-D8-3S4U-7Z:LRTBGVSR4U4VJW8A8BD83S4U7Z, B.Cu at (73.6, 105.6)
- added D57: LED_RGB, LRTBGVSR-4U4V-JW+8A8B-D8-3S4U-7Z:LRTBGVSR4U4VJW8A8BD83S4U7Z, B.Cu at (73.6, 110.6)
- added D58: LED_RGB, LRTBGVSR-4U4V-JW+8A8B-D8-3S4U-7Z:LRTBGVSR4U4VJW8A8BD83S4U7Z, B.Cu at (73.6, 115.6)
- added D59: LED_RGB, LRTBGVSR-4U4V-JW+8A8B-D8-3S4U-7Z:LRTBGVSR4U4VJW8A8BD83S4U7Z, B.Cu at (73.6, 120.6)
- added D6: LED_RGB, LRTBGVSR-4U4V-JW+8A8B-D8-3S4U-7Z:LRTBGVSR4U4VJW8A8BD83S4U7Z, B.Cu at (58.6, 95.6)
- added D60: LED_RGB, LRTBGVSR-4U4V-JW+8A8B-D8-3S4U-7Z:LRTBGVSR4U4VJW8A8BD83S4U7Z, B.Cu at (73.6, 125.6)
- added D61: LED_RGB, LRTBGVSR-4U4V-JW+8A8B-D8-3S4U-7Z:LRTBGVSR4U4VJW8A8BD83S4U7Z, B.Cu at (73.6, 130.6)
- added D62: LED_RGB, LRTBGVSR-4U4V-JW+8A8B-D8-3S4U-7Z:LRTBGVSR4U4VJW8A8BD83S4U7Z, B.Cu at (73.6, 135.6)
- added D63: LED_RGB, LRTBGVSR-4U4V-JW+8A8B-D8-3S4U-7Z:LRTBGVSR4U4VJW8A8BD83S4U7Z, B.Cu at (73.6, 140.6)
- added D64: LED_RGB, LRTBGVSR-4U4V-JW+8A8B-D8-3S4U-7Z:LRTBGVSR4U4VJW8A8BD83S4U7Z, B.Cu at (73.6, 145.6)
- added D65: LED_RGB, LRTBGVSR-4U4V-JW+8A8B-D8-3S4U-7Z:LRTBGVSR4U4VJW8A8BD83S4U7Z, B.Cu at (78.6, 70.6)
- added D66: LED_RGB, LRTBGVSR-4U4V-JW+8A8B-D8-3S4U-7Z:LRTBGVSR4U4VJW8A8BD83S4U7Z, B.Cu at (78.6, 75.6)
- added D67: LED_RGB, LRTBGVSR-4U4V-JW+8A8B-D8-3S4U-7Z:LRTBGVSR4U4VJW8A8BD83S4U7Z, B.Cu at (78.6, 80.6)
- added D68: LED_RGB, LRTBGVSR-4U4V-JW+8A8B-D8-3S4U-7Z:LRTBGVSR4U4VJW8A8BD83S4U7Z, B.Cu at (78.6, 85.6)
- added D69: LED_RGB, LRTBGVSR-4U4V-JW+8A8B-D8-3S4U-7Z:LRTBGVSR4U4VJW8A8BD83S4U7Z, B.Cu at (78.6, 90.6)
- added D7: LED_RGB, LRTBGVSR-4U4V-JW+8A8B-D8-3S4U-7Z:LRTBGVSR4U4VJW8A8BD83S4U7Z, B.Cu at (58.6, 100.6)
- added D70: LED_RGB, LRTBGVSR-4U4V-JW+8A8B-D8-3S4U-7Z:LRTBGVSR4U4VJW8A8BD83S4U7Z, B.Cu at (78.6, 95.6)
- added D71: LED_RGB, LRTBGVSR-4U4V-JW+8A8B-D8-3S4U-7Z:LRTBGVSR4U4VJW8A8BD83S4U7Z, B.Cu at (78.6, 100.6)
- added D72: LED_RGB, LRTBGVSR-4U4V-JW+8A8B-D8-3S4U-7Z:LRTBGVSR4U4VJW8A8BD83S4U7Z, B.Cu at (78.6, 105.6)
- added D73: LED_RGB, LRTBGVSR-4U4V-JW+8A8B-D8-3S4U-7Z:LRTBGVSR4U4VJW8A8BD83S4U7Z, B.Cu at (78.6, 110.6)
- added D74: LED_RGB, LRTBGVSR-4U4V-JW+8A8B-D8-3S4U-7Z:LRTBGVSR4U4VJW8A8BD83S4U7Z, B.Cu at (78.6, 115.6)
- added D75: LED_RGB, LRTBGVSR-4U4V-JW+8A8B-D8-3S4U-7Z:LRTBGVSR4U4VJW8A8BD83S4U7Z, B.Cu at (78.6, 120.6)
- added D76: LED_RGB, LRTBGVSR-4U4V-JW+8A8B-D8-3S4U-7Z:LRTBGVSR4U4VJW8A8BD83S4U7Z, B.Cu at (78.6, 125.6)
- added D77: LED_RGB, LRTBGVSR-4U4V-JW+8A8B-D8-3S4U-7Z:LRTBGVSR4U4VJW8A8BD83S4U7Z, B.Cu at (78.6, 130.6)
- added D78: LED_RGB, LRTBGVSR-4U4V-JW+8A8B-D8-3S4U-7Z:LRTBGVSR4U4VJW8A8BD83S4U7Z, B.Cu at (78.6, 135.6)
- added D79: LED_RGB, LRTBGVSR-4U4V-JW+8A8B-D8-3S4U-7Z:LRTBGVSR4U4VJW8A8BD83S4U7Z, B.Cu at (78.6, 140.6)
- added D8: LED_RGB, LRTBGVSR-4U4V-JW+8A8B-D8-3S4U-7Z:LRTBGVSR4U4VJW8A8BD83S4U7Z, B.Cu at (58.6, 105.6)
- added D80: LED_RGB, LRTBGVSR-4U4V-JW+8A8B-D8-3S4U-7Z:LRTBGVSR4U4VJW8A8BD83S4U7Z, B.Cu at (78.6, 145.6)
- added D81: LED_RGB, LRTBGVSR-4U4V-JW+8A8B-D8-3S4U-7Z:LRTBGVSR4U4VJW8A8BD83S4U7Z, B.Cu at (83.6, 70.6)
- added D82: LED_RGB, LRTBGVSR-4U4V-JW+8A8B-D8-3S4U-7Z:LRTBGVSR4U4VJW8A8BD83S4U7Z, B.Cu at (83.6, 75.6)
- added D83: LED_RGB, LRTBGVSR-4U4V-JW+8A8B-D8-3S4U-7Z:LRTBGVSR4U4VJW8A8BD83S4U7Z, B.Cu at (83.6, 80.6)
- added D84: LED_RGB, LRTBGVSR-4U4V-JW+8A8B-D8-3S4U-7Z:LRTBGVSR4U4VJW8A8BD83S4U7Z, B.Cu at (83.6, 85.6)
- added D85: LED_RGB, LRTBGVSR-4U4V-JW+8A8B-D8-3S4U-7Z:LRTBGVSR4U4VJW8A8BD83S4U7Z, B.Cu at (83.6, 90.6)
- added D86: LED_RGB, LRTBGVSR-4U4V-JW+8A8B-D8-3S4U-7Z:LRTBGVSR4U4VJW8A8BD83S4U7Z, B.Cu at (83.6, 95.6)
- added D87: LED_RGB, LRTBGVSR-4U4V-JW+8A8B-D8-3S4U-7Z:LRTBGVSR4U4VJW8A8BD83S4U7Z, B.Cu at (83.6, 100.6)
- added D88: LED_RGB, LRTBGVSR-4U4V-JW+8A8B-D8-3S4U-7Z:LRTBGVSR4U4VJW8A8BD83S4U7Z, B.Cu at (83.6, 105.6)
- added D89: LED_RGB, LRTBGVSR-4U4V-JW+8A8B-D8-3S4U-7Z:LRTBGVSR4U4VJW8A8BD83S4U7Z, B.Cu at (83.6, 110.6)
- added D9: LED_RGB, LRTBGVSR-4U4V-JW+8A8B-D8-3S4U-7Z:LRTBGVSR4U4VJW8A8BD83S4U7Z, B.Cu at (58.6, 110.6)
- added D90: LED_RGB, LRTBGVSR-4U4V-JW+8A8B-D8-3S4U-7Z:LRTBGVSR4U4VJW8A8BD83S4U7Z, B.Cu at (83.6, 115.6)
- added D91: LED_RGB, LRTBGVSR-4U4V-JW+8A8B-D8-3S4U-7Z:LRTBGVSR4U4VJW8A8BD83S4U7Z, B.Cu at (83.6, 120.6)
- added D92: LED_RGB, LRTBGVSR-4U4V-JW+8A8B-D8-3S4U-7Z:LRTBGVSR4U4VJW8A8BD83S4U7Z, B.Cu at (83.6, 125.6)
- added D93: LED_RGB, LRTBGVSR-4U4V-JW+8A8B-D8-3S4U-7Z:LRTBGVSR4U4VJW8A8BD83S4U7Z, B.Cu at (83.6, 130.6)
- added D94: LED_RGB, LRTBGVSR-4U4V-JW+8A8B-D8-3S4U-7Z:LRTBGVSR4U4VJW8A8BD83S4U7Z, B.Cu at (83.6, 135.6)
- added D95: LED_RGB, LRTBGVSR-4U4V-JW+8A8B-D8-3S4U-7Z:LRTBGVSR4U4VJW8A8BD83S4U7Z, B.Cu at (83.6, 140.6)
- added D96: LED_RGB, LRTBGVSR-4U4V-JW+8A8B-D8-3S4U-7Z:LRTBGVSR4U4VJW8A8BD83S4U7Z, B.Cu at (83.6, 145.6)
- added D97: LED_RGB, LRTBGVSR-4U4V-JW+8A8B-D8-3S4U-7Z:LRTBGVSR4U4VJW8A8BD83S4U7Z, B.Cu at (88.6, 70.6)
- added D98: LED_RGB, LRTBGVSR-4U4V-JW+8A8B-D8-3S4U-7Z:LRTBGVSR4U4VJW8A8BD83S4U7Z, B.Cu at (88.6, 75.6)
- added D99: LED_RGB, LRTBGVSR-4U4V-JW+8A8B-D8-3S4U-7Z:LRTBGVSR4U4VJW8A8BD83S4U7Z, B.Cu at (88.6, 80.6)
- added R1: 10k, Resistor_SMD:R_0603_1608Metric, F.Cu at (155.9, 113.7)
- added R2: 37.4k, Resistor_SMD:R_0603_1608Metric, F.Cu at (155.9, 116.2)
- added R3: 10k, Resistor_SMD:R_0603_1608Metric, F.Cu at (155.9, 118.8)
- added R4: 10k, Resistor_SMD:R_0603_1608Metric, F.Cu at (155.9, 121.3)
- added R5: 26.1k, Resistor_SMD:R_0603_1608Metric, F.Cu at (159.9, 111.2)
- added R6: 10k, Resistor_SMD:R_0603_1608Metric, F.Cu at (159.9, 113.7)
- added R7: R, Resistor_SMD:R_0603_1608Metric, F.Cu at (98.0, 98.8)
- added U1: TPS562202, Package_TO_SOT_SMD:SOT-563, F.Cu at (163.3, 124.2)
- added U2: LP5891MRRFR, ul_LP5891MRRFR:VQFN76_RRF_TEX, F.Cu at (99.0, 90.6)
- added U3: TPS562202, Package_TO_SOT_SMD:SOT-563, F.Cu at (163.3, 127.4)
Routing:
- net /LINE0: track 0.00 -> 192.0 mm, vias 0 -> 1
- net /LINE15: track 0.00 -> 187.4 mm, vias 0 -> 1
- net /LINE14: track 0.00 -> 183.4 mm, vias 0 -> 1
- net /R15: track 0.00 -> 181.7 mm, vias 0 -> 16
- net /LINE12: track 0.00 -> 179.8 mm, vias 0 -> 1
- net /LINE13: track 0.00 -> 179.4 mm, vias 0 -> 1
- net /LINE1: track 0.00 -> 177.0 mm, vias 0 -> 1
- net /B15: track 0.00 -> 176.8 mm, vias 0 -> 16
- net /LINE11: track 0.00 -> 175.8 mm, vias 0 -> 1
- net /G15: track 0.00 -> 174.9 mm, vias 0 -> 17
- net /LINE2: track 0.00 -> 172.4 mm, vias 0 -> 1
- net /LINE10: track 0.00 -> 171.8 mm, vias 0 -> 1
- net /LINE9: track 0.00 -> 170.0 mm, vias 0 -> 1
- net /LINE3: track 0.00 -> 167.7 mm, vias 0 -> 1
- net /B14: track 0.00 -> 166.6 mm, vias 0 -> 16
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- added copper zone on In1.Cu, net GND
Other:
- board outline added: 82 x 82 mm
- copper layers 2 -> 4
